File: XOrduino-v1.brd (EAGLE design)
At the start: 81.3 x 53.3 mm, 55 parts, among them J1 10x1F-H8.5, J2 8x1F-H8.5, J3 8x1F-H8.5, J4 6x1F-H8.5, J5 2.5mm, J6 2.5mm, J7 2.5mm, J8 2.5mm, U1 ATMEGA32U4-XUAU, U10 10k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

Commit message: XOrduino v4. Updated silkscreen, shorting jumpers for sensor lines; tweak USB-B.
Parts:
- added U$5: OSHW-LOGOL, SparkFun-Aesthetics:OSHW-LOGO-L
- JP6: device jumper:JP7Q -> xorduino:JP7QS
- X2: value USB-MB-H -> USB; device SparkFun-Connectors:USB-MB-H -> xorduino:USB-MB-H2
Routing:
- net A4: track 41.0 -> 47.3 mm
- net A5: track 46.0 -> 41.1 mm, vias 1 -> 2
- net SOUND: track 48.4 -> 52.7 mm, vias 1 -> 3
Other:
- board text added: "2012-06-08 v4"
- board text added: "XOrduino!"
- board text added: "v4"
- board text removed: "2012-06-08 v3"
- board text removed: "X2"
- board text removed: "v3"
