File: XOrduino-v1.sch (EAGLE design)
At the start: 55 parts, among them J1 10x1F-H8.5, J2 8x1F-H8.5, J3 8x1F-H8.5, J4 6x1F-H8.5, J5 2.5mm, J6 2.5mm, J7 2.5mm, J8 2.5mm, U1 ATMEGA32U4-XUAU, U10 10k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

Commit message: XOrduino v4. Updated silkscreen, shorting jumpers for sensor lines; tweak USB-B.
Parts:
- added U$5: OSHW-LOGOL, SparkFun-Aesthetics:OSHW-LOGOL
- JP6: device jumper:JP7QE -> xorduino:JP7QES
- X2: value USB-MB-H -> USB; device SparkFun-Connectors:USB-MB-H -> xorduino:USB
Changed lines of the file:
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@@
 <layer number="23" name="tOrigins" color="15" fill="1" visible="no" active="no"/>
 <layer number="24" name="bOrigins" color="15" fill="1" visible="no" active="no"/>
-<layer number="25" name="tNames" color="7" fill="1" visible="no" active="no"/>
+<layer number="25" name="tNames" color="5" fill="1" visible="no" active="no"/>
 <layer number="26" name="bNames" color="7" fill="1" visible="no" active="no"/>
 <layer number="27" name="tValues" color="7" fill="1" visible="no" active="no"/>
@@
 <layer number="97" name="Info" color="7" fill="1" visible="yes" active="yes"/>
 <layer number="98" name="Guide" color="6" fill="1" visible="yes" active="yes"/>
-<layer number="100" name="Muster" color="7" fill="1" visible="no" active="yes"/>
+<layer number="100" name="Muster" color="7" fill="1" visible="yes" active="yes"/>
 <layer number="101" name="Patch_Top" color="7" fill="1" visible="no" active="yes"/>
 <layer number="102" name="Vscore" color="7" fill="1" visible="no" active="yes"/>
@@
 <part name="U$1" library="MyPOW" deviceset="+5V" device=""/>
 <part name="X1" library="SparkFun-Connectors" deviceset="USB" device="PCB"/>
-<part name="X2" library="SparkFun-Connectors" deviceset="USB" device="-MB-H"/>
+<part name="X2" library="xorduino" deviceset="USB" device=""/>
 <part name="U$2" library="MyPOW" deviceset="+5V" device=""/>
 <part name="Y1" library="SparkFun-FreqCtrl" deviceset="CRYSTAL" device="HC49US" value="16MHz"/>
@@
 <part name="GND24" library="SparkFun" deviceset="GND" device=""/>
 <part name="C13" library="SparkFun-Passives" deviceset="CAP" device="PTH" value="0.33uF"/>
-<part name="JP6" library="jumper" deviceset="JP7QE" device="" value="Sensor Routing"/>
+<part name="JP6" library="xorduino" deviceset="JP7QES" device="" value="Sensor Routing"/>
 <part name="GND25" library="supply1" deviceset="GND" device=""/>
 <part name="GND26" library="supply1" deviceset="GND" device=""/>
+<part name="U$5" library="SparkFun-Aesthetics" deviceset="OSHW-LOGO" device="L"/>
 </parts>
 <sheets>
@@
 <text x="-120.142" y="-31.496" size="1.27" layer="97">optional</text>
 <text x="169.926" y="43.434" size="1.27" layer="97">optional</text>
-<text x="189.23" y="-58.928" size="2.54" layer="97">3</text>
+<text x="189.23" y="-58.928" size="2.54" layer="97">4</text>
 <text x="192.024" y="-69.088" size="2.54" layer="97">CSA</text>
 <text x="40.64" y="30.48" size="3.81" layer="94" ratio="10" rot="MR0">Scratch Sensor Board</text>
@@
 <instance part="JP6" gate="-6" x="218.44" y="68.58" rot="R270"/>
 <instance part="JP6" gate="-7" x="218.44" y="78.74" rot="R270"/>
+<instance part="U$5" gate="G$1" x="215.9" y="165.1"/>
 </instances>
 <busses>
